File: output/pcbs/left.kicad_pcb (KiCad board)
At the start: 2 copper layers, 138.1 x 100 mm, 66 parts

Commit message: config changes, route pcbs
Parts:
- added H1: , mounting_hole, F.Cu at (95.0, 84.0)
- added H2: , mounting_hole, F.Cu at (209.0, 84.0)
- added H3: , mounting_hole, F.Cu at (95.0, 140.0)
- added H4: , mounting_hole, F.Cu at (188.1, 141.0)
- moved T1 0.50 mm to (214.0, 64.5)
Connections:
- D12 pad 1: P104 -> P010
- D13 pad 1: P106 -> P115
- D17 pad 1: P104 -> P010
- D18 pad 1: P106 -> P115
- D2 pad 1: P104 -> P010
- D22 pad 1: P104 -> P010
- D23 pad 1: P106 -> P115
- D27 pad 1: P104 -> P010
- D28 pad 1: P106 -> P115
- D3 pad 1: P106 -> P115
- D7 pad 1: P104 -> P010
- D8 pad 1: P106 -> P115
- S1 pad 1: P006 -> P106
- S11 pad 1: P017 -> P009
- S12 pad 1: P017 -> P009
- S13 pad 1: P017 -> P009
- S14 pad 1: P017 -> P009
- S15 pad 1: P017 -> P009
- S2 pad 1: P006 -> P106
- S21 pad 1: P022 -> P111
- S22 pad 1: P022 -> P111
- S23 pad 1: P022 -> P111
- S24 pad 1: P022 -> P111
- S25 pad 1: P022 -> P111
- S3 pad 1: P006 -> P106
- S4 pad 1: P006 -> P106
- S5 pad 1: P006 -> P106
