File: output/pcbs/right.kicad_pcb (KiCad board)
At the start: 2 copper layers, 133.3 x 100 mm, 62 parts

Commit message: config changes, route pcbs
Parts:
- added H1: , mounting_hole, F.Cu at (264.0, 84.0)
- added H2: , mounting_hole, F.Cu at (369.0, 84.0)
- added H3: , mounting_hole, F.Cu at (295.0, 141.0)
- added H4: , mounting_hole, F.Cu at (364.0, 141.0)
- moved T1 0.50 mm to (269.0, 64.5)
Connections:
- S10 pad 1: P017 -> P113
- S11 pad 1: P017 -> P113
- S12 pad 1: P020 -> P111
- S13 pad 1: P020 -> P111
- S14 pad 1: P020 -> P111
- S15 pad 1: P020 -> P111
- S16 pad 1: P020 -> P111
- S17 pad 1: P022 -> P009
- S18 pad 1: P022 -> P009
- S19 pad 1: P022 -> P009
- S20 pad 1: P022 -> P009
- S21 pad 1: P022 -> P009
- S7 pad 1: P017 -> P113
- S8 pad 1: P017 -> P113
- S9 pad 1: P017 -> P113
